File: RubiksCubeSolverBoard/RubiksCubeSolverBoard.kicad_sch (KiCad schematic)
At the start: 43 parts, among them J1 Power +12V, J10 MS3, J11 MS1, J12 Power +12V, J13 MS2, J14 MS3, J15 Motor2, J16 MS1, J17 MS2, J18 MS3, J19 Motor3, J2 Power +3.3V, J20 MS1, J21 MS2, J22 MS3, J23 Motor4, J24 MS1, J25 MS2, J26 MS3, J27 Motor5, J28 color sensor, J29 color sensor, J3 MS1, J4 BootOption, J6 SilentBoot, J7 Motor1, J8 Uart, J9 MS2, U1 ESP32-WROOM-32E

Commit message: 2 layer pcb
Parts:
- removed C5: 100uF, Capacitor_THT:CP_Radial_D6.3mm_P2.50mm, symbol Device:C_Polarized
- removed J1: Power +12V, Connector_PinHeader_2.54mm:PinHeader_1x02_P2.54mm_Vertical, symbol Connector:Conn_01x02_Pin
- removed J11: MS1, Connector_PinHeader_2.54mm:PinHeader_1x02_P2.54mm_Vertical, symbol Connector:Conn_01x02_Pin
- removed J14, J18, J22, J26: MS3, Connector_PinHeader_2.54mm:PinHeader_1x02_P2.54mm_Vertical, symbol Connector:Conn_01x02_Pin
- removed J15: Motor2, CustomParts:JST_B5B-XH-A_LF__SN_, symbol CustomParts:B5B-XH-A_LF__SN_
- removed J19: Motor3, CustomParts:JST_B5B-XH-A_LF__SN_, symbol CustomParts:B5B-XH-A_LF__SN_
- removed J2: Power +3.3V, Connector_PinHeader_2.54mm:PinHeader_1x02_P2.54mm_Vertical, symbol Connector:Conn_01x02_Pin
- removed J23: Motor4, CustomParts:JST_B5B-XH-A_LF__SN_, symbol CustomParts:B5B-XH-A_LF__SN_
- removed J27: Motor5, CustomParts:JST_B5B-XH-A_LF__SN_, symbol CustomParts:B5B-XH-A_LF__SN_
- removed J28: color sensor, Connector_PinHeader_2.54mm:PinHeader_1x02_P2.54mm_Vertical, symbol Connector:Conn_01x02_Pin
- removed J29: color sensor, Connector_PinHeader_2.54mm:PinHeader_1x03_P2.54mm_Vertical, symbol Connector:Conn_01x03_Pin
- removed J4: BootOption, Connector_PinHeader_2.54mm:PinHeader_1x02_P2.54mm_Vertical, symbol Connector:Conn_01x02_Pin
- removed U1: ESP32-WROOM-32E, CustomParts:ESP32-WROOM-32E, symbol ESP32-WROOM-32E:ESP32-WROOM-32E
- added C11, C12: 10uF, Capacitor_THT:CP_Radial_D5.0mm_P2.00mm, symbol Device:C_Polarized
- added C5: 0.1uF, Capacitor_SMD:C_0805_2012Metric, symbol Device:C
- added C9: 100uF, Capacitor_THT:CP_Radial_D6.3mm_P2.50mm, symbol Device:C_Polarized
- added D2: LED, LED_SMD:LED_1206_3216Metric_Pad1.42x1.75mm_HandSolder, symbol Device:LED
- added J1: colorSensor, CustomParts:JST_B5B-XH-A_LF__SN_, symbol CustomParts:B5B-XH-A_LF__SN_
- added J14: Motor2, CustomParts:JST_B5B-XH-A_LF__SN_, symbol CustomParts:B5B-XH-A_LF__SN_
- added J15, J19, J23: MS1, Connector_PinHeader_2.54mm:PinHeader_1x02_P2.54mm_Vertical, symbol Connector:Conn_01x02_Pin
- added J18: Motor3, CustomParts:JST_B5B-XH-A_LF__SN_, symbol CustomParts:B5B-XH-A_LF__SN_
- added J2: power, Connector_PinHeader_2.54mm:PinHeader_1x02_P2.54mm_Vertical, symbol Connector:Conn_01x02_Socket
- added J22: Motor4, CustomParts:JST_B5B-XH-A_LF__SN_, symbol CustomParts:B5B-XH-A_LF__SN_
- added J26: Motor5, CustomParts:JST_B5B-XH-A_LF__SN_, symbol CustomParts:B5B-XH-A_LF__SN_
- added R2: 10k, Resistor_SMD:R_0805_2012Metric, symbol Device:R
- added R3: 220Ohm, Resistor_SMD:R_0805_2012Metric, symbol Device:R
- added R4: 0, Resistor_SMD:R_0805_2012Metric, symbol Device:R
- added SW1: reset, Button_Switch_SMD:SW_Push_SPST_NO_Alps_SKRK, symbol Switch:SW_Push
- added SW2: flash, Button_Switch_SMD:SW_Push_SPST_NO_Alps_SKRK, symbol Switch:SW_Push
- added U2: ESP32-WROOM-32E, RF_Module:ESP32-WROOM-32D, symbol RF_Module:ESP32-WROOM-32E
- added VR2: TS1117BCW33_RPG, CustomParts:VREG_TS1117BCW33_RPG, symbol CustomParts:TS1117BCW33_RPG
- J12: value Power +12V -> MS2
- J13, J17, J21, J25: value MS2 -> MS3
- J16, J20, J24: value MS1 -> MS2
- J6: value SilentBoot -> MS1
- R1: footprint Resistor_SMD:R_1206_3216Metric -> Resistor_SMD:R_0805_2012Metric
Connections:
- net +12V: now also C11.1, C9.1, J2.1 (Pin_1), VR2.3 (INPUT); no longer J12.1 (Pin_1)
- net +3.3V: now also J12.2 (Pin_2), J6.2 (Pin_2), C12.1, D2.2 (A), J1.4, J15.2 (Pin_2), J19.2 (Pin_2), J23.2 (Pin_2), R2.1, U2.2 (VDD), VR2.2 (OUTPUT)
- net GND: now also C11.2, C12.2, C5.1, C9.2, J1.5, J2.2 (Pin_2), R3.2, SW1.1, SW2.2, U2.1 (GND), U2.15 (GND), U2.38 (GND), U2.39 (GND), VR2.1 (FIXED/ADJ); no longer J12.2 (Pin_2), J6.2 (Pin_2)
- net at A3.12 (MS3): now also J17.1 (Pin_1)
- net at A3.10 (MS1): now also J15.1 (Pin_1); no longer J16.1 (Pin_1)
- net at A4.11 (MS2): now also J20.1 (Pin_1); no longer J21.1 (Pin_1)
- net at J6.1 (Pin_1): now also A2.10 (MS1)
- net EN: now reaches C3.1, R1.1
- net EN: now also R4.1, U2.3 (EN)
- net RX: now reaches J8.2 (Pin_2)
- net RX: now also U2.34 (RXD0/IO3)
- net TX: now reaches J8.3 (Pin_3)
- net TX: now also U2.35 (TXD0/IO1)
- net at A3.11 (MS2): now also J16.1 (Pin_1); no longer J17.1 (Pin_1)
- net at A4.3 (1B): now also J22.1
- net at A4.4 (1A): now also J22.2
- net at A4.5 (2A): now also J22.4
- net at A4.6 (2B): now also J22.5
- net at A2.12 (MS3): now also J13.1 (Pin_1)
- net at A5.3 (1B): now also J26.1
- net at A5.4 (1A): now also J26.2
- net at A5.5 (2A): now also J26.4
- net at A5.6 (2B): now also J26.5
- net at A4.10 (MS1): now also J19.1 (Pin_1); no longer J20.1 (Pin_1)
- net at A4.12 (MS3): now also J21.1 (Pin_1)
- net at A5.10 (MS1): now also J23.1 (Pin_1); no longer J24.1 (Pin_1)
- net at J25.1 (Pin_1): now also A5.12 (MS3); no longer A5.11 (MS2)
- net at A3.3 (1B): now also J18.1
- net at A3.4 (1A): now also J18.2
- net at A3.5 (2A): now also J18.4
- net at A3.6 (2B): now also J18.5
- net at A2.3 (1B): now also J14.1
- net at A2.4 (1A): now also J14.2
- net at A2.5 (2A): now also J14.4
- net at A2.6 (2B): now also J14.5
- net at A2.11 (MS2): now also J12.1 (Pin_1); no longer J13.1 (Pin_1)
- net IO16 renamed motor1Step
- net motor1Step: now also U2.30 (IO18)
- net IO17 renamed motor2Step
- net motor2Step: now also U2.16 (IO13)
- net IO32 renamed motor3Step
- net motor3Step: now also U2.9 (IO33)
- net IO33 renamed motor3Dir
- net motor3Dir: now also U2.8 (IO32)
- net IO34 renamed motor4Step
- net motor4Step: now also U2.10 (IO25)
- net IO35 renamed motor4Dir
- net motor4Dir: now also U2.11 (IO26)
- net IO36 renamed motor5Dir
- net motor5Dir: now also U2.13 (IO14)
- net IO39 renamed motor5Step
- net motor5Step: now also U2.12 (IO27)
- net IO4 renamed motor1Dir
- net motor1Dir: now also U2.26 (IO4)
- net IO5 renamed motor2Dir
- net motor2Dir: now also U2.23 (IO15)
- new net: C5.2, R4.2, SW1.2
- new net: D2.1 (K), R3.1
- new net: R2.2, U2.27 (IO16)
- new net: A5.11 (MS2), J24.1 (Pin_1)
- new net SCL: J1.3, U2.36 (IO22)
- new net SDA: J1.2, U2.33 (IO21)
- new net boot: SW2.1, U2.25 (IO0)
- new net colorSensorLed: J1.1, U2.31 (IO19)
- no-connect marks 26 -> 19
Other:
- note added: "power"
- note added: "power input"
- moved on the sheet: A1, C1, C2, C3, C4, J10, J3, J8, J9, R1

Commit message: pcb v1.1
Parts:
- removed J10, J13, J17, J21, J25: MS3, Connector_PinHeader_2.54mm:PinHeader_1x02_P2.54mm_Vertical, symbol Connector:Conn_01x02_Pin
- removed J12, J16, J20, J24, J9: MS2, Connector_PinHeader_2.54mm:PinHeader_1x02_P2.54mm_Vertical, symbol Connector:Conn_01x02_Pin
- removed J15, J19, J23, J3, J6: MS1, Connector_PinHeader_2.54mm:PinHeader_1x02_P2.54mm_Vertical, symbol Connector:Conn_01x02_Pin
- removed J2: power, Connector_PinHeader_2.54mm:PinHeader_1x02_P2.54mm_Vertical, symbol Connector:Conn_01x02_Socket
- removed R4: 0, Resistor_SMD:R_0805_2012Metric, symbol Device:R
- added J10: power, Easyeda2kicad:CONN-TH_DB301V-3.5-2P-GN, symbol Connector:Screw_Terminal_01x02
- added J3: M1_StepType, Connector_PinHeader_2.54mm:PinHeader_2x03_P2.54mm_Vertical, symbol Connector_Generic:Conn_02x03_Odd_Even
- added J4: M2_StepType, Connector_PinHeader_2.54mm:PinHeader_2x03_P2.54mm_Vertical, symbol Connector_Generic:Conn_02x03_Odd_Even
- added J5: M3_StepType, Connector_PinHeader_2.54mm:PinHeader_2x03_P2.54mm_Vertical, symbol Connector_Generic:Conn_02x03_Odd_Even
- added J6, J9: M4_StepType, Connector_PinHeader_2.54mm:PinHeader_2x03_P2.54mm_Vertical, symbol Connector_Generic:Conn_02x03_Odd_Even
- C11, C12: footprint Capacitor_THT:CP_Radial_D5.0mm_P2.00mm -> Capacitor_SMD:CP_Elec_4x5.4
- C4, C6, C7, C8, C9: footprint Capacitor_THT:CP_Radial_D6.3mm_P2.50mm -> Capacitor_SMD:CP_Elec_6.3x7.7
Connections:
- net +12V: now also J10.2 (Pin_2)
- net +3.3V: now also J3.1 (Pin_1), J3.3 (Pin_3), J3.5 (Pin_5), J4.1 (Pin_1), J4.3 (Pin_3), J4.5 (Pin_5), J5.1 (Pin_1), J5.3 (Pin_3), J5.5 (Pin_5), J6.1 (Pin_1), J6.3 (Pin_3), J6.5 (Pin_5), J9.1 (Pin_1), J9.3 (Pin_3), J9.5 (Pin_5)
- net EN: now also C5.2, SW1.2
- net GND: now also J10.1 (Pin_1)
- net M5ST3: now reaches A5.12 (MS3)
- net M5ST3: now also J9.2 (Pin_2)
- net M2ST2: now reaches A2.11 (MS2)
- net M2ST2: now also J4.4 (Pin_4)
- net M4ST1: now reaches A4.10 (MS1)
- net M4ST1: now also J6.6 (Pin_6)
- net M4ST2: now reaches A4.11 (MS2)
- net M4ST2: now also J6.4 (Pin_4)
- net M4ST3: now reaches A4.12 (MS3)
- net M4ST3: now also J6.2 (Pin_2)
- net at A4.3 (1B): now also J22.2; no longer J22.1
- net at A4.4 (1A): now also J22.3; no longer J22.2
- net M1ST2: now reaches A1.11 (MS2)
- net M1ST2: now also J3.4 (Pin_4)
- net M2ST1: now reaches A2.10 (MS1)
- net M2ST1: now also J4.6 (Pin_6)
- net M2ST3: now reaches A2.12 (MS3)
- net M2ST3: now also J4.2 (Pin_2)
- net at A2.3 (1B): now also J14.2; no longer J14.1
- net at A2.4 (1A): now also J14.3; no longer J14.2
- net M1ST1: now reaches A1.10 (MS1)
- net M1ST1: now also J3.6 (Pin_6)
- net M3ST3: now reaches A3.12 (MS3)
- net M3ST3: now also J5.2 (Pin_2)
- net M1ST3: now reaches A1.12 (MS3)
- net M1ST3: now also J3.2 (Pin_2)
- net at A1.3 (1B): now also J7.2; no longer J7.1
- net at A1.4 (1A): now also J7.3; no longer J7.2
- net M3ST1: now reaches A3.10 (MS1)
- net M3ST1: now also J5.6 (Pin_6)
- net M3ST2: now reaches A3.11 (MS2)
- net M3ST2: now also J5.4 (Pin_4)
- net at A3.3 (1B): now also J18.2; no longer J18.1
- net at A3.4 (1A): now also J18.3; no longer J18.2
- net M5ST1: now reaches A5.10 (MS1)
- net M5ST1: now also J9.6 (Pin_6)
- net M5ST2: now reaches A5.11 (MS2)
- net M5ST2: now also J9.4 (Pin_4)
- net at A5.3 (1B): now also J26.2; no longer J26.1
- net at A5.4 (1A): now also J26.3; no longer J26.2
